Commit message: add tf for lidar

File: src/patrol_description/urdf/model.urdf (robot description, URDF)
Before this commit: robot robot, 1 links, 0 joints
Links:
- link base_link: geometry collision mesh filename=package://patrol_description/meshes/body2.STL scale=0.001 0.001 0.001; visual mesh filename=package://patrol_description/meshes/body2.STL scale=0.001 0.001 0.001
