File: electronic/MAIN_PCB/main_pcb.sch (EAGLE design)
At the start: 10 parts, among them J5 D1, J6 D2, J7 UART3, T1 2N2222

Commit message: add main pcb
Parts:
- added J8: UART1, SparkFun-Connectors:CONN_04
- added J9: (no value), SparkFun-Connectors:CONN_04
- added U1, U2: (no value), SparkFun-IC-Power:V_REG_LM1117SOT223
- J1, J2, J3, J4, J5, J6: device SparkFun-Connectors:CONN_04JST-PTH -> SparkFun-Connectors:CONN_04POLAR
Connections:
- new net +5V: U$1.5V, U$1.5V2, U1.IN, U2.IN
- new net N$12: J8.4, U$1.11
- new net N$13: J8.3, U$1.12
- new net N$14: J9.4, U$1.23
- new net N$15: J9.3, U$1.22
- new net N$16: J9.2, U$1.21
- new net N$17: J9.1, U$1.20
- net +3V3: now also J8.1, U1.OUT, U1.OUT@1, U2.OUT, U2.OUT@1
- net GND: now also J8.2, U1.ADJ, U2.ADJ
Other:
- moved on the sheet: J7
