File: electronic/COMMUATOR_POWER_PCB/power_pcb.sch (EAGLE design)
At the start: 9 parts, among them IC1 L293D, K1 CB1A-P-12V, K2 CB1A-P-12V

Commit message: change power pcb
Parts:
- removed IC1: L293D, st-microelectronics:L293D
- removed K1: CB1A-P-12V, relay:CB1A-P-12V
- removed U1: (no value), SparkFun-IC-Power:V_REG_LM1117SOT223
- added D1: 1N4004, diode:1N4004
- added J6: (no value), SparkFun-Connectors:CONN_025MM
- added U$2: 12v, diy-modules:DC-DC-STEP-DOWN-MP1584
- added U$3: usb2, diy-modules:DC-DC-STEP-DOWN-MP1584
- added U$4: USb1, diy-modules:DC-DC-STEP-DOWN-MP1584
- added U$5: Jet2, diy-modules:DC-DC-STEP-DOWN-MP1584
- added U$6: Jet1, diy-modules:DC-DC-STEP-DOWN-MP1584
- added U2: (no value), SparkFun-IC-Power:V_REG_78XXSINK
- J1, J3: device SparkFun-Connectors:BANANA_CONN -> SparkFun-Connectors:CONN_025MM
- J5: device SparkFun-Connectors:CONN_04POLAR -> SparkFun-Connectors:CONN_025MM
Connections:
- removed net +12V: IC1.VCC1, IC1.VCC2, J5.1, U1.IN
- removed net +3V3: IC1.1-2EN, IC1.3-4EN, U1.OUT, U1.OUT@1
- removed net N$1: J1.1, K12.P
- removed net REL1: IC1.1Y, K11.2
- removed net REL2: IC1.3Y, K21.1
- removed net RELIN1: IC1.1A, J5.3
- removed net RELIN2: IC1.3A, J5.4
- new net N$11: D1.C, K21.1, U2.OUT
- new net N$13: J6.2, U2.IN
- new net N$4: J1.1, U$5.OUT+.1, U$5.OUT+.2, U$6.OUT+.1, U$6.OUT+.2
- new net N$5: J1.2, U$5.OUT-.1, U$5.OUT-.2, U$6.OUT-.1, U$6.OUT-.2
- new net N$6: J3.2, U$3.OUT-.1, U$3.OUT-.2, U$4.OUT-.1, U$4.OUT-.2
- new net N$7: J3.1, U$3.OUT+.1, U$3.OUT+.2, U$4.OUT+.1, U$4.OUT+.2
- new net N$8: J5.1, U$2.OUT-.1, U$2.OUT-.2
- new net N$9: J5.2, U$2.OUT+.1, U$2.OUT+.2
- net GND: now also D1.A, U$2.IN-.1, U$2.IN-.2, U$3.IN-.1, U$3.IN-.2, U$4.IN-.1, U$4.IN-.2, U$5.IN-.1, U$5.IN-.2, U$6.IN-.1, U$6.IN-.2, U2.GND; no longer IC1.GND1, IC1.GND2, IC1.GND3, IC1.GND4, J3.1, J5.2, K11.1, U1.ADJ
- net N$2: now also J6.1
- net V+: now also U$2.IN+.1, U$2.IN+.2, U$3.IN+.1, U$3.IN+.2, U$4.IN+.1, U$4.IN+.2, U$5.IN+.1, U$5.IN+.2, U$6.IN+.1, U$6.IN+.2; no longer K12.S
